File: Driverino-Shield.kicad_pcb (KiCad board)
At the start: 2 copper layers, 68.6 x 53.3 mm, 55 parts, among them P1 Power, P10 MOT, P11 HALL, P2 Analog, P3 Digital, P4 Digital, P5 CONN_01X01, P6 CONN_01X01, P7 CONN_01X01, P8 CONN_01X01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

Commit message: Update
Parts:
- added JP2: PinHeader_1x02_P1.27mm_Vertical, Connector_PinHeader_1.27mm:PinHeader_1x02_P1.27mm_Vertical, F.Cu at (149.1, 118.3)
- added REF**: OSHW-Logo_19x20mm_SilkScreen, Symbol:OSHW-Logo_19x20mm_SilkScreen, F.Cu at (146.4, 100.7)
- C3: footprint Driverino-Shield:C_0603_1608Metric -> Capacitor_SMD:C_1206_3216Metric
- C4: footprint Driverino-Shield:C_0603_1608Metric -> Capacitor_SMD:C_0402_1005Metric
- JP1: footprint Driverino-Shield:3JUMPER_0603 -> Connector_PinHeader_1.27mm:PinHeader_1x03_P1.27mm_Vertical
- moved C8 43.9 mm to (135.2, 86.2), turned to 90 degrees
- moved C4 6.96 mm to (122.9, 96.5)
- moved C1 5.73 mm to (128.5, 90.7), turned to 0 degrees
- moved D5 4.40 mm to (133.6, 86.2)
- moved C3 4.17 mm to (122.2, 94.6), turned to 0 degrees
- moved R8 3.82 mm to (131.2, 87.0), turned to 180 degrees
- moved R7 3.81 mm to (131.2, 85.4)
- moved R2 2.90 mm to (133.1, 98.8)
- moved F1 1.85 mm to (132.5, 93.8)
- moved C5 0.90 mm to (125.3, 95.0)
- moved C2 0.64 mm to (124.7, 85.9)
- moved C12 0.38 mm to (116.0, 115.3)
- moved R22 0.38 mm to (118.0, 114.8)
- moved R23 0.38 mm to (118.0, 115.8)
- moved R15 0.25 mm to (169.4, 80.6)
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Connections:
- U1 pad 16: (no net) -> /V
Routing:
- net +3.3V: track 0.00 -> 26.0 mm, vias 0 -> 6
- net /HCN: track 0.00 -> 21.8 mm
- net /HCP: track 0.00 -> 20.3 mm
- net /HBN: track 0.00 -> 19.5 mm
- net /HBP: track 0.00 -> 18.0 mm
- net /HAN: track 0.00 -> 17.2 mm
- net /HAP: track 0.00 -> 15.5 mm
- net Net-(JP1-Pad2): track 0.00 -> 8.10 mm
- net /A1: track 0.00 -> 4.86 mm
- net Net-(D4-Pad2): track 0.00 -> 4.42 mm
- net Net-(D3-Pad2): track 0.00 -> 4.42 mm
- net Net-(D2-Pad2): track 0.00 -> 4.42 mm
- net Net-(D1-Pad2): track 0.00 -> 4.42 mm
- net /8: track 0.00 -> 4.29 mm
- net /7: track 0.00 -> 4.29 mm
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- added copper zone on F.Cu, net +36V
- added copper zone on F.Cu, net /FB
- added copper zone on F.Cu, net /SW
- added copper zone on F.Cu, net /U
- added copper zone on F.Cu, net /V
- added copper zone on F.Cu, net /W
- added copper zone on B.Cu, net GNDPWR
Other:
- board text added: "HALL"

Commit message: Routing completed
Parts:
- JP2: value PinHeader_1x02_P1.27mm_Vertical -> VCC_SEL
- R22, R23: footprint Capacitor_SMD:C_0402_1005Metric -> Resistor_SMD:R_0402_1005Metric
- moved D3 41.3 mm to (134.4, 82.1)
- moved R4 38.9 mm to (131.2, 82.1)
- moved D2 5.36 mm to (168.2, 93.8)
- moved R3 4.58 mm to (165.0, 93.8)
- moved C9 3.69 mm to (160.1, 119.0), turned to 90 degrees
- moved D1 2.85 mm to (168.2, 96.0)
- moved D4 2.80 mm to (168.2, 103.9)
- moved C10 2.35 mm to (118.3, 109.8)
- moved C11 2.35 mm to (118.3, 112.6)
- moved C12 2.35 mm to (118.3, 115.3)
- moved P11 2.35 mm to (116.1, 117.0)
- moved R18 2.35 mm to (120.3, 109.3)
- moved R19 2.35 mm to (120.3, 110.3)
- moved R20 2.35 mm to (120.3, 112.1)
- moved R21 2.35 mm to (120.3, 113.1)
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- renumbered L2 to L1
Connections:
- JP2 pad 2: (no net) -> +5V
- P1 pad 4: (no net) -> +3.3V
- P1 pad 5: (no net) -> +5V
Routing:
- net VCC: track 0.00 -> 82.7 mm, vias 0 -> 4
- net /SLEEP: track 0.00 -> 82.1 mm, vias 0 -> 4
- net +3.3V: track 26.0 -> 95.0 mm, vias 6 -> 9
- net /FAULT: track 0.00 -> 68.2 mm, vias 0 -> 2
- net /DRVOFF: track 0.00 -> 68.2 mm, vias 0 -> 2
- net /A1: track 4.86 -> 72.4 mm, vias 0 -> 4
- net /CS: track 0.00 -> 53.2 mm, vias 0 -> 4
- net /ILIM: track 1.74 -> 49.0 mm, vias 0 -> 2
- net /BRAKE: track 0.00 -> 44.6 mm, vias 0 -> 2
- net /FGOUT: track 1.61 -> 45.5 mm, vias 0 -> 2
- net /11(**/MOSI): track 0.00 -> 41.4 mm, vias 0 -> 2
- net /PWM: track 0.00 -> 39.4 mm, vias 0 -> 2
- net /13(SCK): track 0.00 -> 35.9 mm, vias 0 -> 2
- net /12(MISO): track 4.29 -> 39.5 mm, vias 0 -> 2
- net GND: track 0.00 -> 11.8 mm, vias 0 -> 3
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Other:
- board text added: "+"
- board text added: "+3.3V"
- board text added: "-"
- board text added: "A"
- board text added: "B"
- board text added: "C"
- board text added: "FAULT"
- board text added: "GND"
- board text added: "U"
- board text added: "V"
- board text added: "VCC"
- board text added: "VMOT"
- board text added: "W"
