File: PCB/Driverino-Shield.sch (KiCad schematic (older format))
At the start: 56 parts, among them P1 Power, P10 MOT, P11 HALL, P2 Analog, P3 Digital, P4 Digital, P5 CONN_01X01, P6 CONN_01X01, P7 CONN_01X01, P8 CONN_01X01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

Commit message: Update BOM
Parts:
- C1: Digikey 399-7444-1-ND -> (none); Farnell 2118135RL -> (none); RS 802-9967 -> (none); manf# C1206C226M8RACTU -> (none)
- C10, C11, C12, C4: Digikey 445-6901-1-ND -> (none); Farnell 2210830 -> (none); RS 915-5635 -> (none); manf# CGA2B3X7R1V104K050BB -> (none)
- C2: Digikey P124837CT-ND -> (none); Farnell 3126986 -> (none); manf# EEE-FTV151XAV -> (none); manufacturer1 Panasonic -> (none); mpn1 EEEFTV151XAP -> (none)
- C3: Digikey 445-172483-1-ND -> (none); Farnell 2547055 -> (none); RS 915-5354 -> (none); manf# CGA5L1X7R1V106K160AE -> (none)
- C5, C7: Digikey 311-2082-1-ND -> (none); Farnell 2211179 -> (none); RS 200-6596 -> (none); manf# CC0603KRX7R9BB105 -> (none)
- C6: Digikey 490-4762-1-ND -> (none); Farnell 2470416 -> (none); RS 723-4954 -> (none); manf# GCM155R71H103KA55D -> (none)
- C8, C9: Digikey 445-5666-1-ND -> (none); Farnell 2346967 -> (none); RS 788-2985 -> (none); manf# CGA3E2X7R1H104K080AA -> (none)
- D1: Digikey 475-2486-1-ND -> (none); RS 654-5795 -> (none); manf# LO Q976 -> (none)
- D2: Digikey LBQ39G-N1OO-35-1-ND -> (none); RS 697-3610 -> (none); manf# LB Q39G-N1OO-35-1 -> (none)
- D3: Digikey 475-3442-1-ND -> (none); RS 697-3715 -> (none); manf# LT Q39G-Q1OO-25-1 -> (none)
- D4: Farnell 2463989 -> (none); Manufacturer Kingbright -> OSRAM Opto; Mouser (none) -> 720-LSQ976-NR-1; RS 466-3728 -> (none); manf# KP-1608SRC-PRV -> (none); manufacturer1 OSRAM Opto -> (none); mpn KP-1608SRC-PRV -> LS Q976-NR-1; mpn1 LS Q976-NR-1 -> (none)
- D5: Digikey TSZU52C5V1RGG-ND -> (none); RS 796-5676 -> (none); manf# TSZU52C5V1 RGG -> (none); manufacturer1 Taiwan Semiconductor -> (none); mpn1 BZT52C5V1K RKG -> (none)
- F1: Digikey MF-NSMF020-2CT-ND -> (none); Farnell 1817286 -> (none); RS 647-8279 -> (none); manf# MF-NSMF020-2 -> (none)
- JP1: Digikey SAM10238-ND -> (none); Farnell 2856614 -> (none); RS 180-0478 -> (none); manf# TMS-103-01-G-S -> (none)
- JP2: Digikey SAM12199-ND -> (none); Farnell 2505048 -> (none); RS 180-0534 -> (none); manf# TMS-102-01-G-S -> (none)
- L1: Digikey CBC3225T470KRV -> (none); manf# CBC3225T470KRV -> (none)
- P1, P4: Digikey SSW-108-03-G-S-ND -> (none); RS 180-0432 -> (none); manf# SSW-108-03-G-S -> (none); manufacturer1 Samtec -> (none); mpn1 SSW-108-03-T-S -> (none)
- P10: Digikey 0397730003-ND -> (none); manf# 39773-0003 -> (none)
- P11: Digikey WM1737-ND -> (none); Farnell 1012258 -> (none); RS 279-9241 -> (none); manf# 53047-0810 -> (none)
- P2: Digikey SSW-106-03-G-S-ND -> (none); RS 180-0391 -> (none); manf# SSW-106-03-G-S -> (none); manufacturer1 Samtec -> (none); mpn1 SSW-106-03-T-S -> (none)
- P3: Digikey SSW-110-03-G-S-ND -> (none); Farnell 3661270 -> (none); RS 207-9189 -> (none); manf# SSW-110-03-G-S -> (none); manufacturer1 Samtec -> (none); mpn1 SSW-110-03-T-S -> (none)
- P9: Digikey 0397730002-ND -> (none); manf# 39773-0002 -> (none)
- R1, R13, R3, R5: Digikey 541-3949-1-ND -> (none); RS 678-9875 -> (none); manf# CRCW06031K00FKEAC -> (none)
- R10, R11, R12, R14, R15, R16, R17, R9: Digikey 541-4013-1-ND -> (none); RS 678-9670 -> (none); manf# CRCW06030000Z0EBC -> (none)
- R18, R19, R20, R21, R22, R23: Digikey 541-3958-1-ND -> (none); Farnell 2616725 -> (none); RS 812-1723 -> (none); manf# CRCW040210K0JNEDC -> (none); manufacturer1 Vishay -> (none); mpn1 CRCW040210K0JNEDIF -> (none)
- R2, R4, R6: Digikey ESR03EZPF5101-ND -> (none); RS 679-0566 -> (none); manf# ESR03EZPF5101 -> (none); manufacturer1 Vishay -> (none); mpn1 CRCW06035K10FKEA -> (none)
- R7: Digikey ERJ-3RBD6202V-ND -> (none); Farnell 2380068 -> (none); RS 810-2306 -> (none); manf# ERJ3RBD6202V -> (none)
- R8: Digikey 311-10.0KHRCT-ND -> (none); Farnell 9238603 -> (none); RS 199-5443 -> (none); manf# RC0603FR-0710KL -> (none)
- U1: manf# PMCT8316Z0TRGFR -> (none)

Commit message: Update BOM
Parts:
- C10, C11, C12, C4: Mouser 810-CGA2B3X7R1V104K -> 810-CGA3E2X7R1H104K; mpn CGA2B3X7R1V104K050BB -> CGA3E2X7R1H104K080AA
- C2: value 150uF -> 120uF; Mouser 667-EEE-FTV151XAV -> 667-EEE-FKV121XSV; mpn EEE-FTV151XAV -> EEE-FKV121XSV
- C3: Manufacturer TDK -> Taiyo Yuden; Mouser 810-CGA5L1X7R1V106KE -> 963-GMK316AB7106KL; mpn CGA5L1X7R1V106K160AE -> GMK316AB7106KL-TR
- C5, C7: Manufacturer Yageo -> TDK; Mouser 603-CC603KRX7R9BB105 -> 810-C1608X7R1V105KAE; mpn CC0603KRX7R9BB105 -> C1608X7R1V105K080AE
Changed lines of the file:
@@
 F 2 "Driverino-Shield:C_0603_1608Metric" H 4513 4675 30  0001 C CNN
 F 3 "" H 4475 4825 60  0000 C CNN
-F 4 "CC0603KRX7R9BB105" H 4475 4825 50  0001 C CNN "mpn"
-F 5 "Yageo" H 4475 4825 50  0001 C CNN "Manufacturer"
-F 6 "603-CC603KRX7R9BB105" H 4475 4825 50  0001 C CNN "Mouser"
+F 4 "C1608X7R1V105K080AE" H 4475 4825 50  0001 C CNN "mpn"
+F 5 "TDK" H 4475 4825 50  0001 C CNN "Manufacturer"
+F 6 "810-C1608X7R1V105KAE" H 4475 4825 50  0001 C CNN "Mouser"
 	1    4475 4825
 	0    1    1    0
@@
 F 2 "Capacitor_SMD:C_1206_3216Metric" H 4113 5300 30  0001 C CNN
 F 3 "" H 4075 5450 60  0000 C CNN
-F 4 "CGA5L1X7R1V106K160AE" H 4075 5450 50  0001 C CNN "mpn"
-F 5 "TDK" H 4075 5450 50  0001 C CNN "Manufacturer"
-F 6 "810-CGA5L1X7R1V106KE" H 4075 5450 50  0001 C CNN "Mouser"
+F 4 "GMK316AB7106KL-TR" H 4075 5450 50  0001 C CNN "mpn"
+F 5 "Taiyo Yuden" H 4075 5450 50  0001 C CNN "Manufacturer"
+F 6 "963-GMK316AB7106KL" H 4075 5450 50  0001 C CNN "Mouser"
 	1    4075 5450
 	-1   0    0    1
@@
 F 2 "Capacitor_SMD:C_0402_1005Metric" H 4513 5300 30  0001 C CNN
 F 3 "" H 4475 5450 60  0000 C CNN
-F 4 "CGA2B3X7R1V104K050BB" H 4475 5450 50  0001 C CNN "mpn"
+F 4 "CGA3E2X7R1H104K080AA" H 4475 5450 50  0001 C CNN "mpn"
 F 5 "TDK" H 4475 5450 50  0001 C CNN "Manufacturer"
-F 6 "810-CGA2B3X7R1V104K" H 4475 5450 50  0001 C CNN "Mouser"
+F 6 "810-CGA3E2X7R1H104K" H 4475 5450 50  0001 C CNN "Mouser"
 	1    4475 5450
 	-1   0    0    1
@@
 P 3800 5450
 F 0 "C2" H 3650 5500 40  0000 R CNN
-F 1 "150uF" H 3650 5450 40  0000 R CNN
+F 1 "120uF" H 3650 5450 40  0000 R CNN
 F 2 "Driverino-Shield:CP_Elec_6.3x7.7" H 3800 5450 60  0001 C CNN
 F 3 "" H 3800 5450 60  0000 C CNN
-F 4 "EEE-FTV151XAV" H 3800 5450 50  0001 C CNN "mpn"
+F 4 "EEE-FKV121XSV" H 3800 5450 50  0001 C CNN "mpn"
 F 5 "Panasonic" H 3800 5450 50  0001 C CNN "Manufacturer"
-F 6 "667-EEE-FTV151XAV" H 3800 5450 50  0001 C CNN "Mouser"
+F 6 "667-EEE-FKV121XSV" H 3800 5450 50  0001 C CNN "Mouser"
 	1    3800 5450
 	1    0    0    -1
@@
 F 2 "Driverino-Shield:C_0603_1608Metric" H 7788 4675 30  0001 C CNN
 F 3 "" H 7750 4825 60  0000 C CNN
-F 4 "CC0603KRX7R9BB105" H 7750 4825 50  0001 C CNN "mpn"
-F 5 "Yageo" H 7750 4825 50  0001 C CNN "Manufacturer"
-F 6 "603-CC603KRX7R9BB105" H 7750 4825 50  0001 C CNN "Mouser"
+F 4 "C1608X7R1V105K080AE" H 7750 4825 50  0001 C CNN "mpn"
+F 5 "TDK" H 7750 4825 50  0001 C CNN "Manufacturer"
+F 6 "810-C1608X7R1V105KAE" H 7750 4825 50  0001 C CNN "Mouser"
 	1    7750 4825
 	0    -1   -1   0
@@
 F 2 "Capacitor_SMD:C_0402_1005Metric" H 13088 6275 30  0001 C CNN
 F 3 "" H 13050 6425 60  0000 C CNN
-F 4 "CGA2B3X7R1V104K050BB" H 13050 6425 50  0001 C CNN "mpn"
+F 4 "CGA3E2X7R1H104K080AA" H 13050 6425 50  0001 C CNN "mpn"
 F 5 "1" H 13050 6425 50  0001 C CNN "DNF"
 F 6 "TDK" H 13050 6425 50  0001 C CNN "Manufacturer"
-F 7 "810-CGA2B3X7R1V104K" H 13050 6425 50  0001 C CNN "Mouser"
+F 7 "810-CGA3E2X7R1H104K" H 13050 6425 50  0001 C CNN "Mouser"
 	1    13050 6425
 	-1   0    0    1
@@
 F 2 "Capacitor_SMD:C_0402_1005Metric" H 13088 6800 30  0001 C CNN
 F 3 "" H 13050 6950 60  0000 C CNN
-F 4 "CGA2B3X7R1V104K050BB" H 13050 6950 50  0001 C CNN "mpn"
+F 4 "CGA3E2X7R1H104K080AA" H 13050 6950 50  0001 C CNN "mpn"
 F 5 "1" H 13050 6950 50  0001 C CNN "DNF"
 F 6 "TDK" H 13050 6950 50  0001 C CNN "Manufacturer"
-F 7 "810-CGA2B3X7R1V104K" H 13050 6950 50  0001 C CNN "Mouser"
+F 7 "810-CGA3E2X7R1H104K" H 13050 6950 50  0001 C CNN "Mouser"
 	1    13050 6950
 	-1   0    0    1
@@
 F 2 "Capacitor_SMD:C_0402_1005Metric" H 13088 7325 30  0001 C CNN
 F 3 "" H 13050 7475 60  0000 C CNN
-F 4 "CGA2B3X7R1V104K050BB" H 13050 7475 50  0001 C CNN "mpn"
+F 4 "CGA3E2X7R1H104K080AA" H 13050 7475 50  0001 C CNN "mpn"
 F 5 "1" H 13050 7475 50  0001 C CNN "DNF"
 F 6 "TDK" H 13050 7475 50  0001 C CNN "Manufacturer"
-F 7 "810-CGA2B3X7R1V104K" H 13050 7475 50  0001 C CNN "Mouser"
+F 7 "810-CGA3E2X7R1H104K" H 13050 7475 50  0001 C CNN "Mouser"
 	1    13050 7475
 	-1   0    0    1
