File: PCB/Driverino-Shield.kicad_pcb (KiCad board)
At the start: 2 copper layers, 68.6 x 53.3 mm, 58 parts, among them P1 Power, P10 MOT, P11 HALL, P2 Analog, P3 Digital, P4 Digital, P5 CONN_01X01, P6 CONN_01X01, P7 CONN_01X01, P8 CONN_01X01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

Commit message: Update to KiCAD version 8.0
Other:
- net class Default removed
